File: UART/Calculator Schematic/Calculator Schematic.kicad_sch (KiCad schematic)
At the start: 6 parts, among them U1 ATmega328P-MM, U2 PCF8574A, U3 RC1602A

Commit message: Modified KiCad Schematic
Connections:
- net Earth: no longer U2.1 (A0), U2.2 (A1), U2.3 (A2), U3.10 (DB3), U3.7 (DB0), U3.8 (DB1), U3.9 (DB2)
- no-connect marks 0 -> 7
Changed lines of the file:
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@@
   (junction (at 114.3 91.44) (diameter 0) (color 0 0 0 0)
   )
-  (junction (at 177.8 96.52) (diameter 0) (color 0 0 0 0)
-  )
   (junction (at 82.55 142.24) (diameter 0) (color 0 0 0 0)
   )
-  (junction (at 177.8 93.98) (diameter 0) (color 0 0 0 0)
-  )
   (junction (at 104.14 52.07) (diameter 0) (color 0 0 0 0)
   )
@@
   (junction (at 139.7 52.07) (diameter 0) (color 0 0 0 0)
   )
-  (junction (at 177.8 99.06) (diameter 0) (color 0 0 0 0)
-  )
   (junction (at 54.61 101.6) (diameter 0) (color 0 0 0 0)
   )
   (junction (at 114.3 52.07) (diameter 0) (color 0 0 0 0)
   )
-  (junction (at 177.8 142.24) (diameter 0) (color 0 0 0 0)
-  )
-  (junction (at 121.92 101.6) (diameter 0) (color 0 0 0 0)
-  )
-  (junction (at 121.92 104.14) (diameter 0) (color 0 0 0 0)
-  )
+  (no_connect (at 127 99.06))
+  (no_connect (at 127 104.14))
+  (no_connect (at 181.61 91.44))
+  (no_connect (at 181.61 99.06))
+  (no_connect (at 181.61 96.52))
+  (no_connect (at 127 101.6))
+  (no_connect (at 181.61 93.98))
   (wire (pts (xy 114.3 52.07) (xy 139.7 52.07))
     (stroke (width 0) (type default))
@@
     (stroke (width 0) (type default))
   )
-  (wire (pts (xy 121.92 99.06) (xy 121.92 101.6))
-    (stroke (width 0) (type default))
-  )
-  (wire (pts (xy 121.92 104.14) (xy 121.92 106.68))
-    (stroke (width 0) (type default))
-  )
-  (wire (pts (xy 121.92 101.6) (xy 127 101.6))
-    (stroke (width 0) (type default))
-  )
   (wire (pts (xy 152.4 91.44) (xy 165.1 91.44))
     (stroke (width 0) (type default))
@@
     (stroke (width 0) (type default))
   )
-  (wire (pts (xy 191.77 142.24) (xy 177.8 142.24))
-    (stroke (width 0) (type default))
-  )
-  (wire (pts (xy 121.92 104.14) (xy 127 104.14))
-    (stroke (width 0) (type default))
-  )
   (wire (pts (xy 152.4 96.52) (xy 170.18 96.52))
     (stroke (width 0) (type default))
@@
     (stroke (width 0) (type default))
   )
-  (wire (pts (xy 177.8 91.44) (xy 177.8 93.98))
-    (stroke (width 0) (type default))
-  )
   (wire (pts (xy 207.01 101.6) (xy 201.93 101.6))
     (stroke (width 0) (type default))
@@
     (stroke (width 0) (type default))
   )
-  (wire (pts (xy 177.8 96.52) (xy 177.8 99.06))
-    (stroke (width 0) (type default))
-  )
   (wire (pts (xy 82.55 55.88) (xy 82.55 52.07))
     (stroke (width 0) (type default))
@@
     (stroke (width 0) (type default))
   )
-  (wire (pts (xy 177.8 99.06) (xy 181.61 99.06))
-    (stroke (width 0) (type default))
-  )
-  (wire (pts (xy 177.8 142.24) (xy 139.7 142.24))
+  (wire (pts (xy 139.7 142.24) (xy 191.77 142.24))
     (stroke (width 0) (type default))
   )
@@
     (stroke (width 0) (type default))
   )
-  (wire (pts (xy 177.8 93.98) (xy 181.61 93.98))
-    (stroke (width 0) (type default))
-  )
   (wire (pts (xy 167.64 86.36) (xy 181.61 86.36))
     (stroke (width 0) (type default))
@@
     (stroke (width 0) (type default))
   )
-  (wire (pts (xy 177.8 96.52) (xy 181.61 96.52))
-    (stroke (width 0) (type default))
-  )
   (wire (pts (xy 139.7 52.07) (xy 191.77 52.07))
     (stroke (width 0) (type default))
@@
     (stroke (width 0) (type default))
   )
-  (wire (pts (xy 127 99.06) (xy 121.92 99.06))
-    (stroke (width 0) (type default))
-  )
   (wire (pts (xy 25.4 101.6) (xy 33.02 101.6))
     (stroke (width 0) (type default))
@@
     (stroke (width 0) (type default))
   )
-  (wire (pts (xy 177.8 99.06) (xy 177.8 142.24))
-    (stroke (width 0) (type default))
-  )
   (wire (pts (xy 191.77 114.3) (xy 191.77 127))
     (stroke (width 0) (type default))
@@
     (stroke (width 0) (type default))
   )
-  (wire (pts (xy 181.61 91.44) (xy 177.8 91.44))
-    (stroke (width 0) (type default))
-  )
-  (wire (pts (xy 177.8 93.98) (xy 177.8 96.52))
-    (stroke (width 0) (type default))
-  )
   (wire (pts (xy 152.4 109.22) (xy 181.61 109.22))
     (stroke (width 0) (type default))
@@
   )
   (wire (pts (xy 104.14 52.07) (xy 104.14 68.58))
-    (stroke (width 0) (type default))
-  )
-  (wire (pts (xy 121.92 101.6) (xy 121.92 104.14))
     (stroke (width 0) (type default))
   )
@@
         )
       )
-    )
-  )
-  (symbol (lib_id "power:Earth") (at 121.92 106.68 0) (unit 1)
-    (in_bom yes) (on_board yes) (dnp no) (fields_autoplaced)
-    (property "Reference" "#PWR03" (at 121.92 113.03 0)
-      (effects (font (size 1.27 1.27)) hide)
-    )
-    (property "Value" "Earth" (at 121.92 110.49 0)
-      (effects (font (size 1.27 1.27)) hide)
-    )
-    (property "Footprint" "" (at 121.92 106.68 0)
-      (effects (font (size 1.27 1.27)) hide)
-    )
-    (property "Datasheet" "~" (at 121.92 106.68 0)
-      (effects (font (size 1.27 1.27)) hide)
-    )
-    (pin "1")
-    (instances
-      (project "Calculator Schematic"
-        (path "/c607de86-5e0a-4b0a-acd3-3b91ea5a1a66"
-          (reference "#PWR03") (unit 1)
-        )
-      )
